File: z802.kicad_pcb (KiCad board)
At the start: 2 copper layers, 81.3 x 79.8 mm, 17 parts, among them J1 IO Control, J2 IO Data, J3 IO Address, J4 Power, SW1 SW_Push, U1 28C256, U2 Z80CPU, U3 74LS32, U4 74LS04, U5 HM62256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

Commit message: Finish PCB.
Routing:
- net Net-(J2-Pad6): track 11.2 -> 162.8 mm, vias 0 -> 11
- net Net-(J3-Pad10): track 12.0 -> 162.9 mm, vias 0 -> 11
- net GND: track 0.00 -> 140.1 mm, vias 0 -> 4
- net WR: track 11.7 -> 142.6 mm, vias 1 -> 5
- net Net-(J2-Pad7): track 10.7 -> 138.2 mm, vias 0 -> 4
- net Net-(J2-Pad4): track 12.2 -> 123.3 mm, vias 0 -> 5
- net Net-(J2-Pad8): track 67.6 -> 171.5 mm, vias 2 -> 6
- net Net-(J2-Pad5): track 11.7 -> 113.0 mm, vias 0 -> 3
- net Net-(J3-Pad14): track 83.7 -> 177.5 mm, vias 0 -> 9
- net Net-(J3-Pad11): track 84.9 -> 152.4 mm, vias 6 -> 18
- net Net-(J3-Pad12): track 101.2 -> 156.8 mm, vias 0 -> 6
- net VCC: track 200.2 -> 252.3 mm, vias 1 -> 4
- net Net-(J3-Pad15): track 88.3 -> 130.3 mm, vias 0 -> 1
- net Net-(J3-Pad13): track 78.0 -> 114.7 mm, vias 0 -> 1
- net Net-(J2-Pad1): track 111.8 -> 147.4 mm, vias 1 -> 5
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- added copper zone on F.Cu, net GND
