File: z802-3.kicad_pcb (KiCad board)
At the start: 2 copper layers, 68.8 x 107.4 mm, 17 parts, among them J1 IO Control, J2 IO Data, J3 IO Address, J4 Power, SW1 SW_Push, U1 28C256, U2 Z80CPU, U3 74LS32, U4 74LS04, U5 HM62256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

Commit message: Re-design PCB for the fourth time.
Routing:
- net WR: track 165.7 -> 160.4 mm, vias 3 -> 2
- net VCC: track 242.9 -> 240.2 mm
Changed lines of the file:
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@@
     (thickness 1.6)
     (drawings 4)
-    (tracks 547)
+    (tracks 542)
     (zones 0)
     (modules 17)
@@
   (segment (start 143.764 135.382) (end 145.288 133.858) (width 0.25) (layer F.Cu) (net 4))
   (segment (start 132.446998 135.382) (end 143.764 135.382) (width 0.25) (layer F.Cu) (net 4))
-  (segment (start 162.798001 177.752001) (end 162.798001 179.232001) (width 0.25) (layer B.Cu) (net 4))
-  (segment (start 161.798 176.752) (end 162.798001 177.752001) (width 0.25) (layer B.Cu) (net 4))
-  (via (at 148.844 168.91) (size 0.8) (drill 0.4) (layers F.Cu B.Cu) (net 4))
-  (segment (start 162.798001 179.232001) (end 162.278001 179.752001) (width 0.25) (layer B.Cu) (net 4))
-  (segment (start 162.278001 179.752001) (end 159.686001 179.752001) (width 0.25) (layer B.Cu) (net 4))
-  (segment (start 159.686001 179.752001) (end 148.844 168.91) (width 0.25) (layer B.Cu) (net 4))
   (via (at 143.256 161.544) (size 0.8) (drill 0.4) (layers F.Cu B.Cu) (net 4))
-  (segment (start 148.844 168.91) (end 143.256 163.322) (width 0.25) (layer F.Cu) (net 4))
-  (segment (start 143.256 163.322) (end 143.256 161.544) (width 0.25) (layer F.Cu) (net 4))
   (segment (start 141.732 137.414) (end 145.288 133.858) (width 0.25) (layer B.Cu) (net 4))
   (segment (start 143.256 153.811002) (end 139.082999 149.638001) (width 0.25) (layer B.Cu) (net 4))
@@
   (segment (start 143.256 161.544) (end 143.256 153.811002) (width 0.25) (layer B.Cu) (net 4))
   (segment (start 141.732 144.272) (end 141.732 137.414) (width 0.25) (layer B.Cu) (net 4))
+  (segment (start 156.686 176.752) (end 161.798 176.752) (width 0.25) (layer F.Cu) (net 4))
+  (segment (start 143.256 161.544) (end 143.256 163.322) (width 0.25) (layer F.Cu) (net 4))
+  (segment (start 143.256 163.322) (end 156.686 176.752) (width 0.25) (layer F.Cu) (net 4))
   (segment (start 125.476 76.708) (end 118.11 84.074) (width 0.25) (layer F.Cu) (net 5))
   (segment (start 118.11 84.074) (end 107.188 84.074) (width 0.25) (layer F.Cu) (net 5))
@@
   (segment (start 152.146 163.068) (end 145.796 169.418) (width 0.25) (layer B.Cu) (net 30))
   (segment (start 152.146 152.146) (end 152.146 163.068) (width 0.25) (layer B.Cu) (net 30))
-  (segment (start 125.984 150.114) (end 124.968 149.098) (width 0.25) (layer B.Cu) (net 30))
-  (segment (start 125.984 159.315002) (end 125.984 150.114) (width 0.25) (layer B.Cu) (net 30))
   (segment (start 140.97 169.418) (end 136.086998 169.418) (width 0.25) (layer B.Cu) (net 30))
-  (segment (start 136.086998 169.418) (end 125.984 159.315002) (width 0.25) (layer B.Cu) (net 30))
   (segment (start 129.54 169.418) (end 136.086998 169.418) (width 0.25) (layer B.Cu) (net 30))
   (segment (start 125.222 173.736) (end 129.54 169.418) (width 0.25) (layer B.Cu) (net 30))
@@
   (segment (start 152.146 148.59) (end 152.146 152.146) (width 0.25) (layer B.Cu) (net 30))
   (segment (start 153.271001 147.464999) (end 152.146 148.59) (width 0.25) (layer B.Cu) (net 30))
+  (segment (start 125.984 150.114) (end 124.968 149.098) (width 0.25) (layer B.Cu) (net 30))
+  (segment (start 129.54 169.418) (end 125.984 165.862) (width 0.25) (layer B.Cu) (net 30))
+  (segment (start 125.984 165.862) (end 125.984 150.114) (width 0.25) (layer B.Cu) (net 30))
   (segment (start 142.494 129.032) (end 137.668 133.858) (width 0.25) (layer F.Cu) (net 31))
   (segment (start 144.018 129.032) (end 142.494 129.032) (width 0.25) (layer F.Cu) (net 31))
