File: z802.sch (KiCad schematic (older format))
At the start: 17 parts, among them J1 IO Control, J2 IO Data, J3 IO Address, J4 Power, SW1 SW_Push, U1 28C256, U2 Z80CPU, U3 74LS32, U4 74LS04, U5 HM62256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

Commit message: Re-design PCB.
Parts:
- J1: footprint Connector_PinHeader_1.27mm:PinHeader_1x03_P1.27mm_Vertical -> Connector_PinHeader_2.00mm:PinHeader_1x03_P2.00mm_Vertical
- J2: footprint Connector_PinHeader_1.27mm:PinHeader_1x08_P1.27mm_Vertical -> Connector_PinHeader_2.00mm:PinHeader_1x08_P2.00mm_Vertical
- J3: footprint Connector_PinHeader_1.27mm:PinHeader_1x16_P1.27mm_Vertical -> Connector_PinHeader_2.00mm:PinHeader_1x16_P2.00mm_Vertical
- J4: footprint Connector_PinHeader_1.27mm:PinHeader_1x02_P1.27mm_Vertical -> Connector_PinHeader_2.00mm:PinHeader_1x02_P2.00mm_Vertical
Changed lines of the file:
@@
 F 0 "J1" H 1158 3981 50  0000 C CNN
 F 1 "IO Control" H 1158 3890 50  0000 C CNN
-F 2 "Connector_PinHeader_1.27mm:PinHeader_1x03_P1.27mm_Vertical" H 1050 3700 50  0001 C CNN
+F 2 "Connector_PinHeader_2.00mm:PinHeader_1x03_P2.00mm_Vertical" H 1050 3700 50  0001 C CNN
 F 3 "~" H 1050 3700 50  0001 C CNN
 	1    1050 3700
@@
 F 0 "J2" H 1158 4931 50  0000 C CNN
 F 1 "IO Data" H 1158 4840 50  0000 C CNN
-F 2 "Connector_PinHeader_1.27mm:PinHeader_1x08_P1.27mm_Vertical" H 1050 4450 50  0001 C CNN
+F 2 "Connector_PinHeader_2.00mm:PinHeader_1x08_P2.00mm_Vertical" H 1050 4450 50  0001 C CNN
 F 3 "~" H 1050 4450 50  0001 C CNN
 	1    1050 4450
@@
 F 0 "J3" H 1158 7481 50  0000 C CNN
 F 1 "IO Address" H 1158 7390 50  0000 C CNN
-F 2 "Connector_PinHeader_1.27mm:PinHeader_1x16_P1.27mm_Vertical" H 1050 6600 50  0001 C CNN
+F 2 "Connector_PinHeader_2.00mm:PinHeader_1x16_P2.00mm_Vertical" H 1050 6600 50  0001 C CNN
 F 3 "~" H 1050 6600 50  0001 C CNN
 	1    1050 6600
@@
 F 0 "J4" H 9208 5031 50  0000 C CNN
 F 1 "Power" H 9208 4940 50  0000 C CNN
-F 2 "Connector_PinHeader_1.27mm:PinHeader_1x02_P1.27mm_Vertical" H 9100 4850 50  0001 C CNN
+F 2 "Connector_PinHeader_2.00mm:PinHeader_1x02_P2.00mm_Vertical" H 9100 4850 50  0001 C CNN
 F 3 "~" H 9100 4850 50  0001 C CNN
 	1    9100 4850

Commit message: Re-design PCB for the fourth time.
Parts:
- added unit 5 of U3
- added unit 7 of U4
- J1: footprint Connector_PinHeader_2.00mm:PinHeader_1x03_P2.00mm_Vertical -> Connector_PinHeader_2.54mm:PinHeader_1x03_P2.54mm_Vertical
- J2: footprint Connector_PinHeader_2.00mm:PinHeader_1x08_P2.00mm_Vertical -> Connector_PinHeader_2.54mm:PinHeader_1x08_P2.54mm_Vertical
- J3: footprint Connector_PinHeader_2.00mm:PinHeader_1x16_P2.00mm_Vertical -> Connector_PinHeader_2.54mm:PinHeader_1x16_P2.54mm_Vertical
- J4: footprint Connector_PinHeader_2.00mm:PinHeader_1x02_P2.00mm_Vertical -> Connector_PinHeader_2.54mm:PinHeader_1x02_P2.54mm_Vertical
Connections:
- net GND: now also U3.7 (GND), U4.7 (GND)
- net VCC: now also U3.14 (VCC), U4.14 (VCC)
Other:
- moved on the sheet: J4

Commit message: Redesign the PCB for the 6th time.
Parts:
- removed J1: IO Control, Connector_PinHeader_2.54mm:PinHeader_1x03_P2.54mm_Vertical, symbol Connector:Conn_01x03_Male
- added C1, C2, C3, C4, C5: 0.1u, Capacitor_THT:C_Disc_D8.0mm_W2.5mm_P5.00mm, symbol Device:C_Small
- added C6: 10u, Capacitor_THT:C_Disc_D8.0mm_W2.5mm_P5.00mm, symbol Device:C_Small
- added J1: IO Control, Connector_PinHeader_2.54mm:PinHeader_1x04_P2.54mm_Vertical, symbol Connector:Conn_01x04_Male
- D1: value LED -> LED M1
- U3, U4: footprint (none) -> Package_DIP:DIP-14_W7.62mm
Connections:
- net GND: now also C1.2, C2.2, C3.2, C4.2, C5.2, C6.2
- net IOREQ: now also J1.1 (Pin_1)
- net RD: now also J1.3 (Pin_3)
- net VCC: now also C1.1, C2.1, C3.1, C4.1, C5.1, C6.1
- net WAIT: now also J1.4 (Pin_4)
- net WR: now also J1.2 (Pin_2)
Other:
- note added: "Power"
- moved on the sheet: J4, R1, R2, R3, R4, U3E, U4G
